Commit message: add link1 and link2

File: install/kr210_description/share/kr210_description/urdf/kr210_arm.urdf.xacro (robot description, xacro)
@@ -7,8 +7,24 @@
             <mesh filename="package://kr210_description/meshes/kr210l150/visual/base_link.dae"/>
         </geometry>
-        <origin xyz="0 0 0" rpy="0 0 0"/>
+        <origin xyz="0 0 0" rpy="-${pi/2} 0 0"/>
         <material name="">
             <color rgba="0.75294 0.75294 0.75294 1"/>
         </material>
+    </visual>
+</link>
+<link name="link_1">
+    <visual>
+        <geometry>
+            <mesh filename="package://kr210_description/meshes/kr210l150/visual/link_1.dae"/>
+        </geometry>
+        <origin xyz="0 0 0" rpy="0 0 0"/>
+    </visual>
+</link>
+<link name="link_2">
+    <visual>
+        <geometry>
+            <mesh filename="package://kr210_description/meshes/kr210l150/visual/link_2.dae"/>
+        </geometry>
+        <origin xyz="0 0 0" rpy="-${pi/2} 0 0"/>
     </visual>
 </link>
@@ -18,3 +34,15 @@
     <origin xyz="0 0 0" rpy="0 0 0"/>
 </joint>
+<joint name="joint_1" type="revolute">
+    <parent link="base_link"/>
+    <child link="link_1"/>
+    <origin xyz="0 0 0.33" rpy="0 0 0"/>
+    <axis xyz="0 0 1"/>
+    <limit lower="${-185.0 * (pi / 180.0)}" upper="${185.0 * (pi / 180.0)}" effort="300" velocity="${123.0 * (pi / 180.0)}"/>
+</joint>
+<joint name="joint_2" type="fixed">
+    <parent link="link_1"/>
+    <child link="link_2"/>
+    <origin xyz="0.35 0 0.42" rpy="0 0 0"/>
+</joint>
 </robot>

Commit message: add joint 3 and joint 4

File: install/kr210_description/share/kr210_description/urdf/kr210_arm.urdf.xacro (robot description, xacro)
@@ -29,4 +29,20 @@
     </visual>
 </link>
+<link name="link_3">
+    <visual>
+        <geometry>
+            <mesh filename="package://kr210_description/meshes/kr210l150/visual/link_3.dae"/>
+        </geometry>
+        <origin xyz="0 -0.184 0" rpy="${-pi/2} 0 0"/>
+    </visual>
+</link>
+<link name="link_4">
+    <visual>
+        <geometry>
+            <mesh filename="package://kr210_description/meshes/kr210l150/visual/link_4.dae"/>
+        </geometry>
+        <origin xyz="0 0 0" rpy="0 0 0"/>
+    </visual>
+</link>
 <joint name="fixed_base_joint" type="fixed">
     <parent link="base_footprint"/>
@@ -41,8 +57,24 @@
     <limit lower="${-185.0 * (pi / 180.0)}" upper="${185.0 * (pi / 180.0)}" effort="300" velocity="${123.0 * (pi / 180.0)}"/>
 </joint>
-<joint name="joint_2" type="fixed">
+<joint name="joint_2" type="revolute">
     <parent link="link_1"/>
     <child link="link_2"/>
     <origin xyz="0.35 0 0.42" rpy="0 0 0"/>
+    <axis xyz="0 1 0"/>
+    <limit lower="${-45*pi/180}" upper="${85*pi/180}" effort="300" velocity="${115*pi/180}"/>
+</joint>
+<joint name="joint_3" type="revolute">
+    <parent link="link_2"/>
+    <child link="link_3"/>
+    <origin xyz="0 0 1.25" rpy="0 0 0"/>
+    <axis xyz="0 1 0"/>
+    <limit lower="${-210*pi/180}" upper="${65*pi/180}" effort="300" velocity="${112 * pi/180}"/>
+</joint>
+<joint name="joint_4" type="revolute">
+    <parent link="link_3"/>
+    <child link="link_4"/>
+    <origin xyz="0.96 0 -0.054" rpy="0 0 0"/>
+    <axis xyz="1 0 0"/>
+    <limit lower="${-125 * pi/180}" upper="${125*pi/180}" effort="300" velocity="${179*pi/180}"/>
 </joint>
 </robot>

Commit message: finished all joint visual

File: install/kr210_description/share/kr210_description/urdf/kr210_arm.urdf.xacro (robot description, xacro)
@@ -42,4 +42,20 @@
             <mesh filename="package://kr210_description/meshes/kr210l150/visual/link_4.dae"/>
         </geometry>
+        <origin xyz="0 0 0" rpy="${-pi/2} 0 0"/>
+    </visual>
+</link>
+<link name="link_5">
+    <visual>
+        <geometry>
+            <mesh filename="package://kr210_description/meshes/kr210l150/visual/link_5.dae"/>
+        </geometry>
+        <origin xyz="0 0 0" rpy="${-pi/2} 0 0"/>
+    </visual>
+</link>
+<link name="link_6">
+    <visual>
+        <geometry>
+            <mesh filename="package://kr210_description/meshes/kr210l150/visual/link_6.dae"/>
+        </geometry>
         <origin xyz="0 0 0" rpy="0 0 0"/>
     </visual>
@@ -78,3 +94,17 @@
     <limit lower="${-125 * pi/180}" upper="${125*pi/180}" effort="300" velocity="${179*pi/180}"/>
 </joint>
+<joint name="joint_5" type="revolute">
+    <parent link="link_4"/>
+    <child link="link_5"/>
+    <origin xyz="0.54 0 0" rpy="0 0 0"/>
+    <axis xyz="0 1 0"/>
+    <limit lower="${-125 * pi/180}" upper="${125*pi/180}" effort="300" velocity="${172*pi/180}"/>
+</joint>
+<joint name="joint_6" type="revolute">
+    <parent link="link_5"/>
+    <child link="link_6"/>
+    <origin xyz="0.193 0 0" rpy="0 0 0"/>
+    <axis xyz="1 0 0"/>
+    <limit lower="${-350*pi/180}" upper="${350*pi/180}" effort="300" velocity="${219*pi/180}"/>
+</joint>
 </robot>

Commit message: add collision to links

File: install/kr210_description/share/kr210_description/urdf/kr210_arm.urdf.xacro (robot description, xacro)
@@ -12,4 +12,10 @@
         </material>
     </visual>
+    <collision>
+        <geometry>
+            <mesh filename="package://kr210_description/meshes/kr210l150/collision/base_link.stl"/>
+        </geometry>
+        <origin xyz="0 0 0" rpy="${-pi/2} 0 0"/>
+    </collision>
 </link>
 <link name="link_1">
@@ -20,4 +26,10 @@
         <origin xyz="0 0 0" rpy="0 0 0"/>
     </visual>
+    <collision>
+        <geometry>
+            <mesh filename="package://kr210_description/meshes/kr210l150/collision/link_1.stl"/>
+        </geometry>
+        <origin xyz="0 0 0" rpy="0 0 0"/>
+    </collision>
 </link>
 <link name="link_2">
@@ -28,4 +40,10 @@
         <origin xyz="0 0 0" rpy="-${pi/2} 0 0"/>
     </visual>
+    <collision>
+        <geometry>
+            <mesh filename="package://kr210_description/meshes/kr210l150/collision/link_2.stl"/>
+        </geometry>
+        <origin xyz="0 0 0" rpy="0 0 0"/>
+    </collision>
 </link>
 <link name="link_3">
@@ -36,4 +54,10 @@
         <origin xyz="0 -0.184 0" rpy="${-pi/2} 0 0"/>
     </visual>
+    <collision>
+        <geometry>
+            <mesh filename="package://kr210_description/meshes/kr210l150/collision/link_3.stl"/>
+        </geometry>
+        <origin xyz="0 -0.184 0" rpy="0 0 0"/>
+    </collision>
 </link>
 <link name="link_4">
@@ -44,4 +68,10 @@
         <origin xyz="0 0 0" rpy="${-pi/2} 0 0"/>
     </visual>
+    <collision>
+        <geometry>
+            <mesh filename="package://kr210_description/meshes/kr210l150/collision/link_4.stl"/>
+        </geometry>
+        <origin xyz="0 0 0" rpy="0 0 0"/>
+    </collision>
 </link>
 <link name="link_5">
@@ -52,4 +82,10 @@
         <origin xyz="0 0 0" rpy="${-pi/2} 0 0"/>
     </visual>
+    <collision>
+        <geometry>
+            <mesh filename="package://kr210_description/meshes/kr210l150/collision/link_5.stl"/>
+        </geometry>
+        <origin xyz="0 0 0" rpy="0 0 0"/>
+    </collision>
 </link>
 <link name="link_6">
@@ -60,4 +96,10 @@
         <origin xyz="0 0 0" rpy="0 0 0"/>
     </visual>
+    <collision>
+        <geometry>
+            <mesh filename="package://kr210_description/meshes/kr210l150/collision/link_6.stl"/>
+        </geometry>
+        <origin xyz="0 0 0" rpy="0 0 0"/>
+    </collision>
 </link>
 <joint name="fixed_base_joint" type="fixed">

Commit message: remove and rebuild

File: install/kr210_description/share/kr210_description/urdf/kr210_arm.urdf.xacro (robot description, xacro)
@@ -154,4 +154,12 @@
     </inertial>
 </link>
+<link name="gripper_link">
+    <visual>
+        <geometry>
+            <mesh filename="file://$(find kr210_description)/meshes/gripper/gripper_base.dae"/>
+        </geometry>
+        <origin xyz="0 0 0" rpy="0 0 0"/>
+    </visual>
+</link>
 <joint name="fixed_base_joint" type="fixed">
     <parent link="base_footprint"/>
@@ -207,3 +215,8 @@
     <dynamics friction="1000" damping="1000"/>
 </joint>
+<joint name="gripper_joint">
+    <parent link="link_6"/>
+    <child link="gripper_link"/>
+    <orgin xyz="0 0 0" rpy="0 0 0"/>
+</joint>
 </robot>

Commit message: add finger gripper

File: install/kr210_description/share/kr210_description/urdf/kr210_arm.urdf.xacro (robot description, xacro)
@@ -8,13 +8,4 @@
 <xacro:property name="mass5" value="7"/>
 <xacro:property name="mass6" value="0.5"/>
-<xacro:macro name="box_inertia" params="m l w h xyz rpy">
-        <inertial>
-            <origin xyz="${xyz}" rpy="${rpy}"/>
-            <mass value="${m}" />
-            <inertia ixx="${(m/12) * (h*h + l*l)}" ixy="0" ixz="0"
-                     iyy="${(m/12) * (w*w + l*l)}" iyz="0"
-                     izz="${(m/12) * (w*w + h*h)}"/>
-        </inertial>
-    </xacro:macro>
 <link name="base_footprint"/>
 <link name="base_link">
@@ -24,7 +15,4 @@
         </geometry>
         <origin xyz="0 0 0" rpy="-${pi/2} 0 0"/>
-        <material name="">
-            <color rgba="0.75294 0.75294 0.75294 1"/>
-        </material>
     </visual>
     <collision>
@@ -37,5 +25,5 @@
         <mass value="${base_mass}"/>
         <inertia ixx="60" iyy="0" izz="0" ixy="70" ixz="0" iyz="100" />
-        <orgin xyz="0 0 0" rpy="0 0 0"/>
+        <origin xyz="0 0 0" rpy="0 0 0"/>
     </inertial>
 </link>
@@ -162,4 +150,41 @@
     </visual>
 </link>
+<link name="right_finger_link">
+    <visual>
+        <geometry>
+            <mesh filename="file://$(find kr210_description)/meshes/gripper/finger_right.dae"/>
+        </geometry>
+        <origin xyz="0 0 0" rpy="0 0 0"/>
+    </visual>
+</link>
+<link name="left_finger_link">
+    <visual>
+        <geometry>
+            <mesh filename="file://$(find kr210_description)/meshes/gripper/finger_left.dae"/>
+        </geometry>
+        <origin xyz="0 0 0" rpy="0 0 0"/>
+    </visual>
+</link>
+<joint name="gripper_joint" type="fixed">
+    <parent link="link_6"/>
+    <child link="gripper_link"/>
+    <origin xyz="0.11 0 0" rpy="0 0 0"/>
+</joint>
+<joint name="gripper_right_finger_joint" type="prismatic">
+    <parent link="gripper_link"/>
+    <child link="right_finger_link"/>
+    <origin xyz="0.15 -0.0725 0" rpy="0 0 0"/>
+    <axis xyz="0 1 0"/>
+    <limit effort="100" lower="-0.01" upper="0.06" velocity="0.05"/>
+    <dynamics damping="0.7"/>
+</joint>
+<joint name="gripper_left_finger_joint" type="prismatic">
+    <parent link="gripper_link"/>
+    <child link="left_finger_link"/>
+    <origin xyz="0.15 0.0725 0" rpy="0 0 0"/>
+    <axis xyz="0 -1 0"/>
+    <limit effort="100" lower="-0.01" upper="0.06" velocity="0.05"/>
+    <dynamics damping="0.7"/>
+</joint>
 <joint name="fixed_base_joint" type="fixed">
     <parent link="base_footprint"/>
@@ -215,8 +240,3 @@
     <dynamics friction="1000" damping="1000"/>
 </joint>
-<joint name="gripper_joint">
-    <parent link="link_6"/>
-    <child link="gripper_link"/>
-    <orgin xyz="0 0 0" rpy="0 0 0"/>
-</joint>
 </robot>
