Commit message: add transmission to gripper

File: install/kr210_description/share/kr210_description/urdf/kr210_gripper.urdf.xacro (robot description, xacro)
@@ -79,3 +79,23 @@
         <dynamics damping="0.7"/>
     </joint>
+    <transmission name="trans_7">
+        <type>transmission_interface/SimpleTransmission</type>
+        <joint name="gripper_right_finger_joint">
+            <hardwareInterface>hardware_interface/EffortJointInterface</hardwareInterface>
+        </joint>
+        <actuator name="motor_7">
+            <hardwareInterface>hardware_interface/EffortJointInterface</hardwareInterface>
+            <mechanicalReduction>1</mechanicalReduction>
+        </actuator>
+    </transmission>
+    <transmission name="trans_8">
+        <type>transmission_interface/SimpleTransmission</type>
+        <joint name="gripper_left_finger_joint">
+            <hardwareInterface>hardware_interface/EffortJointInterface</hardwareInterface>
+        </joint>
+        <actuator name="motor_8">
+            <hardwareInterface>hardware_interface/EffortJointInterface</hardwareInterface>
+            <mechanicalReduction>1</mechanicalReduction>
+        </actuator>
+    </transmission>
 </robot>
