Commit message: fix gazebo not responding

File: install/kr210_description/share/kr210_description/urdf/kr210.urdf.xacro (robot description, xacro)
@@ -1,5 +1,5 @@
 <?xml version="1.0"?>
 <robot name="kuka" xmlns:xacro="http://www.ros.org/wiki/xacro">
-    <xacro:include filename="kr210_arm_gazebo.urdf.xacro"/>
+    <!-- <xacro:include filename="kr210_arm_gazebo.urdf.xacro"/> -->
     <xacro:include filename="kr210_arm.urdf.xacro"/>
 </robot>

File: install/kr210_description/share/kr210_description/urdf/kr210_arm.urdf.xacro (robot description, xacro)
@@ -1,220 +1,209 @@
 <?xml version="1.0"?>
-<robot name="kuka_arm" xmlns:xacro="http://www.ros.org/wiki/xacro">
-  <!--Define constants-->
-  <xacro:property name="deg" value="0.017453293"/><!--degrees to radians-->
-  <xacro:property name="mass0" value="150" />
-  <xacro:property name="mass1" value="138" />
-  <xacro:property name="mass2" value="95" />
-  <xacro:property name="mass3" value="71" />
-  <xacro:property name="mass4" value="17" />
-  <xacro:property name="mass5" value="7" />
-  <xacro:property name="mass6" value="0.5" />
-  <xacro:property name="gripper_mass" value="0.3" />
-  <xacro:property name="finger_mass" value="0.1" />
-  <xacro:property name="gripper_type" value="two_finger" /><!--value="vacuum" or "two_finger"-->
-  <xacro:property name="vacuum_gripper_radius" value="0.1" />
-  <!--Links-->
-  <link name="base_footprint"/>
-  <link name="base_link">
-    <inertial>
-      <origin xyz="0 0 0" rpy="0 0 0"/>
-      <mass value="${mass0}"/>
-      <inertia ixx="60" ixy="0" ixz="0" iyy="70" iyz="0" izz="100"/>
-    </inertial>
-    <visual>
-      <origin xyz="0 0 0" rpy="${-pi/2} 0 0"/>
-      <geometry>
-        <mesh filename="package://kr210_description/meshes/kr210l150/visual/base_link.dae"/>
-      </geometry>
-      <material name="">
-        <color rgba="0.75294 0.75294 0.75294 1"/>
-      </material>
-    </visual>
-    <collision>
-      <origin xyz="0 0 0" rpy="${-pi/2} 0 0"/>
-      <geometry>
-        <mesh filename="package://kr210_description/meshes/kr210l150/collision/base_link.stl"/>
-      </geometry>
-    </collision>
-  </link>
-  <link name="link_1">
-    <inertial>
-      <origin xyz="0 0 0.4" rpy="0 0 0"/>
-      <mass value="${mass1}"/>
-      <inertia ixx="30" ixy="0" ixz="0" iyy="50" iyz="0" izz="50"/>
-    </inertial>
-    <visual>
-      <origin xyz="0 0 0" rpy="0 0 0"/>
-      <geometry>
-        <mesh filename="package://kr210_description/meshes/kr210l150/visual/link_1.dae"/>
-      </geometry>
-      <material name="">
-        <color rgba="0.75294 0.75294 0.75294 1"/>
-      </material>
-    </visual>
-    <collision>
-      <origin xyz="0 0 0" rpy="0 0 0"/>
-      <geometry>
-        <mesh filename="package://kr210_description/meshes/kr210l150/collision/link_1.stl"/>
-      </geometry>
-    </collision>
-  </link>
-  <link name="link_2">
-    <inertial>
-      <origin xyz="0 0 0.44751" rpy="0 0 0"/>
-      <mass value="${mass2}"/>
-      <inertia ixx="40" ixy="0" ixz="0" iyy="40" iyz="0" izz="10"/>
-    </inertial>
-    <visual>
-      <origin xyz="0 0 0" rpy="${-pi/2} 0 0"/>
-      <geometry>
-        <mesh filename="package://kr210_description/meshes/kr210l150/visual/link_2.dae"/>
-      </geometry>
-      <material name="">
-        <color rgba="0.75294 0.75294 0.75294 1"/>
-      </material>
-    </visual>
-    <collision>
-      <origin xyz="0 0 0" rpy="0 0 0"/>
-      <geometry>
-        <mesh filename="package://kr210_description/meshes/kr210l150/collision/link_2.stl"/>
-      </geometry>
-    </collision>
-  </link>
-  <link name="link_3">
-    <inertial>
-      <origin xyz="0.18842 0.18344 -0.042799" rpy="0 0 0"/>
-      <mass value="${mass3}"/>
-      <inertia ixx="1" ixy="0" ixz="0" iyy="10" iyz="0" izz="10"/>
-    </inertial>
-    <visual>
-      <origin xyz="0 -0.184 0" rpy="${-pi/2} 0 0"/>
-      <geometry>
-        <mesh filename="package://kr210_description/meshes/kr210l150/visual/link_3.dae"/>
-      </geometry>
-      <material name="">
-        <color rgba="0.75294 0.75294 0.75294 1"/>
-      </material>
-    </visual>
-    <collision>
-      <origin xyz="0 -0.184 0" rpy="0 0 0"/>
-      <geometry>
-        <mesh filename="package://kr210_description/meshes/kr210l150/collision/link_3.stl"/>
-      </geometry>
-    </collision>
-  </link>
-  <link name="link_4">
-    <inertial>
-      <origin xyz="0.27146 -0.007326 0" rpy="0 0 0"/>
-      <mass value="${mass4}"/>
-      <inertia ixx="0.18" ixy="0" ixz="0" iyy="0.55" iyz="0" izz="0.64"/>
-    </inertial>
-    <visual>
-      <origin xyz="0 0 0" rpy="${-pi/2} 0 0"/>
-      <geometry>
-        <mesh filename="package://kr210_description/meshes/kr210l150/visual/link_4.dae"/>
-      </geometry>
-      <material name="">
-        <color rgba="0.75294 0.75294 0.75294 1"/>
-      </material>
-    </visual>
-    <collision>
-      <origin xyz="0 0 0" rpy="0 0 0"/>
-      <geometry>
-        <mesh filename="package://kr210_description/meshes/kr210l150/collision/link_4.stl"/>
-      </geometry>
-    </collision>
-  </link>
-  <link name="link_5">
-    <inertial>
-      <origin xyz="0 0 0" rpy="0 0 0"/>
-      <mass value="${mass5}"/>
-      <inertia ixx="0.04" ixy="0" ixz="0" iyy="0.068" iyz="0" izz="0.068"/>
-    </inertial>
-    <visual>
-      <origin xyz="0 0 0" rpy="${-pi/2} 0 0"/>
-      <geometry>
-        <mesh filename="package://kr210_description/meshes/kr210l150/visual/link_5.dae"/>
-      </geometry>
-      <material name="">
-        <color rgba="0.75294 0.75294 0.75294 1"/>
-      </material>
-    </visual>
-    <collision>
-      <origin xyz="0 0 0" rpy="0 0 0"/>
-      <geometry>
-        <mesh filename="package://kr210_description/meshes/kr210l150/collision/link_5.stl"/>
-      </geometry>
-    </collision>
-  </link>
-  <link name="link_6">
-    <inertial>
-      <origin xyz="0 0 0" rpy="0 0 0"/>
-      <mass value="${mass6}"/>
-      <inertia ixx="0.004" ixy="0" ixz="0" iyy="0.003" iyz="0" izz="0.003"/>
-    </inertial>
-    <visual>
-      <origin xyz="0 0 0" rpy="0 0 0"/>
-      <geometry>
-        <mesh filename="package://kr210_description/meshes/kr210l150/visual/link_6.dae"/>
-      </geometry>
-      <material name="">
-        <color rgba="0.75294 0.75294 0.75294 1"/>
-      </material>
-    </visual>
-    <collision>
-      <origin xyz="0 0 0" rpy="0 0 0"/>
-      <geometry>
-        <mesh filename="package://kr210_description/meshes/kr210l150/collision/link_6.stl"/>
-      </geometry>
-    </collision>
-  </link>
-  <!-- joints -->
-  <joint name="fixed_base_joint" type="fixed">
+<robot xmlns:xacro="http://www.ros.org/wiki/xacro">
+<xacro:property name="base_mass" value="150"/>
+<xacro:property name="mass1" value="138"/>
+<xacro:property name="mass2" value="95"/>
+<xacro:property name="mass3" value="71"/>
+<xacro:property name="mass4" value="17"/>
+<xacro:property name="mass5" value="7"/>
+<xacro:property name="mass6" value="0.5"/>
+<xacro:macro name="box_inertia" params="m l w h xyz rpy">
+        <inertial>
+            <origin xyz="${xyz}" rpy="${rpy}"/>
+            <mass value="${m}" />
+            <inertia ixx="${(m/12) * (h*h + l*l)}" ixy="0" ixz="0"
+                     iyy="${(m/12) * (w*w + l*l)}" iyz="0"
+                     izz="${(m/12) * (w*w + h*h)}"/>
+        </inertial>
+    </xacro:macro>
+<link name="base_footprint"/>
+<link name="base_link">
+    <visual>
+        <geometry>
+            <mesh filename="file://$(find kr210_description)/meshes/kr210l150/visual/base_link.dae"/>
+        </geometry>
+        <origin xyz="0 0 0" rpy="-${pi/2} 0 0"/>
+        <material name="">
+            <color rgba="0.75294 0.75294 0.75294 1"/>
+        </material>
+    </visual>
+    <collision>
+        <geometry>
+            <mesh filename="file://$(find kr210_description)/meshes/kr210l150/collision/base_link.stl"/>
+        </geometry>
+        <origin xyz="0 0 0" rpy="${-pi/2} 0 0"/>
+    </collision>
+    <inertial>
+        <mass value="${base_mass}"/>
+        <inertia ixx="60" iyy="0" izz="0" ixy="70" ixz="0" iyz="100" />
+        <orgin xyz="0 0 0" rpy="0 0 0"/>
+    </inertial>
+</link>
+<link name="link_1">
+    <visual>
+        <geometry>
+            <mesh filename="file://$(find kr210_description)/meshes/kr210l150/visual/link_1.dae"/>
+        </geometry>
+        <origin xyz="0 0 0" rpy="0 0 0"/>
+    </visual>
+    <collision>
+        <geometry>
+            <mesh filename="file://$(find kr210_description)/meshes/kr210l150/collision/link_1.stl"/>
+        </geometry>
+        <origin xyz="0 0 0" rpy="0 0 0"/>
+    </collision>
+    <inertial>
+        <mass value="${mass1}"/>
+        <inertia ixx="30" ixy="0" ixz="0" iyy="50" iyz="0" izz="50"/>
+        <origin xyz="0 0 0.4" rpy="0 0 0"/>
+    </inertial>
+</link>
+<link name="link_2">
+    <visual>
+        <geometry>
+            <mesh filename="file://$(find kr210_description)/meshes/kr210l150/visual/link_2.dae"/>
+        </geometry>
+        <origin xyz="0 0 0" rpy="-${pi/2} 0 0"/>
+    </visual>
+    <collision>
+        <geometry>
+            <mesh filename="file://$(find kr210_description)/meshes/kr210l150/collision/link_2.stl"/>
+        </geometry>
+        <origin xyz="0 0 0" rpy="0 0 0"/>
+    </collision>
+    <inertial>
+        <mass value="${mass2}"/>
+        <inertia ixx="40" ixy="0" ixz="0" iyy="40" iyz="0" izz="10"/>
+        <origin xyz="0 0 0" rpy="0 0 0"/>
+    </inertial>
+</link>
+<link name="link_3">
+    <visual>
+        <geometry>
+            <mesh filename="file://$(find kr210_description)/meshes/kr210l150/visual/link_3.dae"/>
+        </geometry>
+        <origin xyz="0 -0.184 0" rpy="${-pi/2} 0 0"/>
+    </visual>
+    <collision>
+        <geometry>
+            <mesh filename="file://$(find kr210_description)/meshes/kr210l150/collision/link_3.stl"/>
+        </geometry>
+        <origin xyz="0 -0.184 0" rpy="0 0 0"/>
+    </collision>
+    <inertial>
+        <mass value="${mass3}"/>
+        <inertia ixx="1" ixy="0" ixz="0" iyy="10" iyz="0" izz="10"/>
+        <origin xyz="0.18842 0.18344 -0.042799" rpy="0 0 0"/>
+    </inertial>
+</link>
+<link name="link_4">
+    <visual>
+        <geometry>
+            <mesh filename="file://$(find kr210_description)/meshes/kr210l150/visual/link_4.dae"/>
+        </geometry>
+        <origin xyz="0 0 0" rpy="${-pi/2} 0 0"/>
+    </visual>
+    <collision>
+        <geometry>
+            <mesh filename="file://$(find kr210_description)/meshes/kr210l150/collision/link_4.stl"/>
+        </geometry>
+        <origin xyz="0 0 0" rpy="0 0 0"/>
+    </collision>
+    <inertial>
+        <mass value="${mass4}"/>
+        <inertia ixx="0.18" ixy="0" ixz="0" iyy="0.55" iyz="0" izz="0.64"/>
+        <origin xyz="0.27146 -0.007326 0" rpy="0 0 0"/>
+    </inertial>
+</link>
+<link name="link_5">
+    <visual>
+        <geometry>
+            <mesh filename="file://$(find kr210_description)/meshes/kr210l150/visual/link_5.dae"/>
+        </geometry>
+        <origin xyz="0 0 0" rpy="${-pi/2} 0 0"/>
+    </visual>
+    <collision>
+        <geometry>
+            <mesh filename="file://$(find kr210_description)/meshes/kr210l150/collision/link_5.stl"/>
+        </geometry>
+        <origin xyz="0 0 0" rpy="0 0 0"/>
+    </collision>
+    <inertial>
+        <mass value="${mass5}"/>
+        <inertia ixx="0.04" ixy="0" ixz="0" iyy="0.068" iyz="0" izz="0.068"/>
+        <origin xyz="0 0 0" rpy="0 0 0"/>
+    </inertial>
+</link>
+<link name="link_6">
+    <visual>
+        <geometry>
+            <mesh filename="file://$(find kr210_description)/meshes/kr210l150/visual/link_6.dae"/>
+        </geometry>
+        <origin xyz="0 0 0" rpy="0 0 0"/>
+    </visual>
+    <collision>
+        <geometry>
+            <mesh filename="file://$(find kr210_description)/meshes/kr210l150/collision/link_6.stl"/>
+        </geometry>
+        <origin xyz="0 0 0" rpy="0 0 0"/>
+    </collision>
+    <inertial>
+        <mass value="${mass6}"/>
+        <inertia ixx="0.004" ixy="0" ixz="0" iyy="0.003" iyz="0" izz="0.003"/>
+        <origin xyz="0 0 0" rpy="0 0 0"/>
+    </inertial>
+</link>
+<joint name="fixed_base_joint" type="fixed">
     <parent link="base_footprint"/>
     <child link="base_link"/>
     <origin xyz="0 0 0" rpy="0 0 0"/>
-  </joint>
-  <joint name="joint_1" type="revolute">
-    <origin xyz="0 0 0.33" rpy="0 0 0"/>
+</joint>
+<joint name="joint_1" type="revolute">
     <parent link="base_link"/>
     <child link="link_1"/>
+    <origin xyz="0 0 0.33" rpy="0 0 0"/>
     <axis xyz="0 0 1"/>
-    <limit lower="${-185*deg}" upper="${185*deg}" effort="300" velocity="${123*deg}"/>
-  </joint>
-  <joint name="joint_2" type="revolute">
-    <origin xyz="0.35 0 0.42" rpy="0 0 0"/>
+    <limit lower="${-185.0 * (pi / 180.0)}" upper="${185.0 * (pi / 180.0)}" effort="300" velocity="${123.0 * (pi / 180.0)}"/>
+    <dynamics friction="1000" damping="1000"/>
+</joint>
+<joint name="joint_2" type="revolute">
     <parent link="link_1"/>
     <child link="link_2"/>
+    <origin xyz="0.35 0 0.42" rpy="0 0 0"/>
     <axis xyz="0 1 0"/>
-    <limit lower="${-45*deg}" upper="${85*deg}" effort="300" velocity="${115*deg}"/>
-  </joint>
-  <joint name="joint_3" type="revolute">
-    <origin xyz="0 0 1.25" rpy="0 0 0"/>
+    <limit lower="${-45*pi/180}" upper="${85*pi/180}" effort="300" velocity="${115*pi/180}"/>
+    <dynamics friction="1000" damping="1000"/>
+</joint>
+<joint name="joint_3" type="revolute">
     <parent link="link_2"/>
     <child link="link_3"/>
+    <origin xyz="0 0 1.25" rpy="0 0 0"/>
     <axis xyz="0 1 0"/>
-    <limit lower="${-210*deg}" upper="${(155-90)*deg}" effort="300" velocity="${112*deg}"/>
-  </joint>
-  <joint name="joint_4" type="revolute">
-    <origin xyz="0.96 0 -0.054" rpy="0 0 0"/>
+    <limit lower="${-210*pi/180}" upper="${65*pi/180}" effort="300" velocity="${112 * pi/180}"/>
+    <dynamics friction="1000" damping="1000"/>
+</joint>
+<joint name="joint_4" type="revolute">
     <parent link="link_3"/>
     <child link="link_4"/>
+    <origin xyz="0.96 0 -0.054" rpy="0 0 0"/>
     <axis xyz="1 0 0"/>
-    <limit lower="${-350*deg}" upper="${350*deg}" effort="300" velocity="${179*deg}"/>
-  </joint>
-  <joint name="joint_5" type="revolute">
-    <origin xyz="0.54 0 0" rpy="0 0 0"/>
+    <limit lower="${-125 * pi/180}" upper="${125*pi/180}" effort="300" velocity="${179*pi/180}"/>
+    <dynamics friction="1000" damping="1000"/>
+</joint>
+<joint name="joint_5" type="revolute">
     <parent link="link_4"/>
     <child link="link_5"/>
+    <origin xyz="0.54 0 0" rpy="0 0 0"/>
     <axis xyz="0 1 0"/>
-    <limit lower="${-125*deg}" upper="${125*deg}" effort="300" velocity="${172*deg}"/>
-  </joint>
-  <joint name="joint_6" type="revolute">
-    <origin xyz="0.193 0 0" rpy="0 0 0"/>
+    <limit lower="${-125 * pi/180}" upper="${125*pi/180}" effort="300" velocity="${172*pi/180}"/>
+    <dynamics friction="1000" damping="1000"/>
+</joint>
+<joint name="joint_6" type="revolute">
     <parent link="link_5"/>
     <child link="link_6"/>
+    <origin xyz="0.193 0 0" rpy="0 0 0"/>
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