Commit message: fix gazebo not responding

File: src/kr210_description/urdf/kr210_arm.urdf.xacro (robot description, xacro)
@@ -8,9 +8,18 @@
 <xacro:property name="mass5" value="7"/>
 <xacro:property name="mass6" value="0.5"/>
+<xacro:macro name="box_inertia" params="m l w h xyz rpy">
+        <inertial>
+            <origin xyz="${xyz}" rpy="${rpy}"/>
+            <mass value="${m}" />
+            <inertia ixx="${(m/12) * (h*h + l*l)}" ixy="0" ixz="0"
+                     iyy="${(m/12) * (w*w + l*l)}" iyz="0"
+                     izz="${(m/12) * (w*w + h*h)}"/>
+        </inertial>
+    </xacro:macro>
 <link name="base_footprint"/>
 <link name="base_link">
     <visual>
         <geometry>
-            <mesh filename="package://kr210_description/meshes/kr210l150/collision/base_link.stl"/>
+            <mesh filename="file://$(find kr210_description)/meshes/kr210l150/visual/base_link.dae"/>
         </geometry>
         <origin xyz="0 0 0" rpy="-${pi/2} 0 0"/>
@@ -21,5 +30,5 @@
     <collision>
         <geometry>
-            <mesh filename="package://kr210_description/meshes/kr210l150/collision/base_link.stl"/>
+            <mesh filename="file://$(find kr210_description)/meshes/kr210l150/collision/base_link.stl"/>
         </geometry>
         <origin xyz="0 0 0" rpy="${-pi/2} 0 0"/>
@@ -27,5 +36,5 @@
     <inertial>
         <mass value="${base_mass}"/>
-        <inertia ixx="60" ixy="0" ixz="0" iyy="70" iyz="0" izz="100"/>
+        <inertia ixx="60" iyy="0" izz="0" ixy="70" ixz="0" iyz="100" />
         <orgin xyz="0 0 0" rpy="0 0 0"/>
     </inertial>
@@ -34,24 +43,24 @@
     <visual>
         <geometry>
-            <mesh filename="package://kr210_description/meshes/kr210l150/visual/link_1.dae"/>
-        </geometry>
-        <origin xyz="0 0 0" rpy="0 0 0"/>
-    </visual>
-    <collision>
-        <geometry>
-            <mesh filename="package://kr210_description/meshes/kr210l150/collision/link_1.stl"/>
-        </geometry>
-        <origin xyz="0 0 0" rpy="0 0 0"/>
-    </collision>
-    <!-- <inertial>
+            <mesh filename="file://$(find kr210_description)/meshes/kr210l150/visual/link_1.dae"/>
+        </geometry>
+        <origin xyz="0 0 0" rpy="0 0 0"/>
+    </visual>
+    <collision>
+        <geometry>
+            <mesh filename="file://$(find kr210_description)/meshes/kr210l150/collision/link_1.stl"/>
+        </geometry>
+        <origin xyz="0 0 0" rpy="0 0 0"/>
+    </collision>
+    <inertial>
         <mass value="${mass1}"/>
         <inertia ixx="30" ixy="0" ixz="0" iyy="50" iyz="0" izz="50"/>
-        <origin xyz="0 0 0" rpy="0 0 0"/>
-    </inertial> -->
+        <origin xyz="0 0 0.4" rpy="0 0 0"/>
+    </inertial>
 </link>
 <link name="link_2">
     <visual>
         <geometry>
-            <mesh filename="package://kr210_description/meshes/kr210l150/visual/link_2.dae"/>
+            <mesh filename="file://$(find kr210_description)/meshes/kr210l150/visual/link_2.dae"/>
         </geometry>
         <origin xyz="0 0 0" rpy="-${pi/2} 0 0"/>
@@ -59,18 +68,18 @@
     <collision>
         <geometry>
-            <mesh filename="package://kr210_description/meshes/kr210l150/collision/link_2.stl"/>
-        </geometry>
-        <origin xyz="0 0 0" rpy="0 0 0"/>
-    </collision>
-    <!-- <inertial>
+            <mesh filename="file://$(find kr210_description)/meshes/kr210l150/collision/link_2.stl"/>
+        </geometry>
+        <origin xyz="0 0 0" rpy="0 0 0"/>
+    </collision>
+    <inertial>
         <mass value="${mass2}"/>
         <inertia ixx="40" ixy="0" ixz="0" iyy="40" iyz="0" izz="10"/>
         <origin xyz="0 0 0" rpy="0 0 0"/>
-    </inertial> -->
+    </inertial>
 </link>
 <link name="link_3">
     <visual>
         <geometry>
-            <mesh filename="package://kr210_description/meshes/kr210l150/visual/link_3.dae"/>
+            <mesh filename="file://$(find kr210_description)/meshes/kr210l150/visual/link_3.dae"/>
         </geometry>
         <origin xyz="0 -0.184 0" rpy="${-pi/2} 0 0"/>
@@ -78,18 +87,18 @@
     <collision>
         <geometry>
-            <mesh filename="package://kr210_description/meshes/kr210l150/collision/link_3.stl"/>
+            <mesh filename="file://$(find kr210_description)/meshes/kr210l150/collision/link_3.stl"/>
         </geometry>
         <origin xyz="0 -0.184 0" rpy="0 0 0"/>
     </collision>
-    <!-- <inertial>
+    <inertial>
         <mass value="${mass3}"/>
         <inertia ixx="1" ixy="0" ixz="0" iyy="10" iyz="0" izz="10"/>
-        <origin xyz="0 0 0" rpy="0 0 0"/>
-    </inertial> -->
+        <origin xyz="0.18842 0.18344 -0.042799" rpy="0 0 0"/>
+    </inertial>
 </link>
 <link name="link_4">
     <visual>
         <geometry>
-            <mesh filename="package://kr210_description/meshes/kr210l150/visual/link_4.dae"/>
+            <mesh filename="file://$(find kr210_description)/meshes/kr210l150/visual/link_4.dae"/>
         </geometry>
         <origin xyz="0 0 0" rpy="${-pi/2} 0 0"/>
@@ -97,18 +106,18 @@
     <collision>
         <geometry>
-            <mesh filename="package://kr210_description/meshes/kr210l150/collision/link_4.stl"/>
-        </geometry>
-        <origin xyz="0 0 0" rpy="0 0 0"/>
-    </collision>
-    <!-- <inertial>
+            <mesh filename="file://$(find kr210_description)/meshes/kr210l150/collision/link_4.stl"/>
+        </geometry>
+        <origin xyz="0 0 0" rpy="0 0 0"/>
+    </collision>
+    <inertial>
         <mass value="${mass4}"/>
         <inertia ixx="0.18" ixy="0" ixz="0" iyy="0.55" iyz="0" izz="0.64"/>
-        <origin xyz="0 0 0" rpy="0 0 0"/>
-    </inertial> -->
+        <origin xyz="0.27146 -0.007326 0" rpy="0 0 0"/>
+    </inertial>
 </link>
 <link name="link_5">
     <visual>
         <geometry>
-            <mesh filename="package://kr210_description/meshes/kr210l150/visual/link_5.dae"/>
+            <mesh filename="file://$(find kr210_description)/meshes/kr210l150/visual/link_5.dae"/>
         </geometry>
         <origin xyz="0 0 0" rpy="${-pi/2} 0 0"/>
@@ -116,32 +125,32 @@
     <collision>
         <geometry>
-            <mesh filename="package://kr210_description/meshes/kr210l150/collision/link_5.stl"/>
-        </geometry>
-        <origin xyz="0 0 0" rpy="0 0 0"/>
-    </collision>
-    <!-- <inertial>
+            <mesh filename="file://$(find kr210_description)/meshes/kr210l150/collision/link_5.stl"/>
+        </geometry>
+        <origin xyz="0 0 0" rpy="0 0 0"/>
+    </collision>
+    <inertial>
         <mass value="${mass5}"/>
         <inertia ixx="0.04" ixy="0" ixz="0" iyy="0.068" iyz="0" izz="0.068"/>
         <origin xyz="0 0 0" rpy="0 0 0"/>
-    </inertial> -->
+    </inertial>
 </link>
 <link name="link_6">
     <visual>
         <geometry>
-            <mesh filename="package://kr210_description/meshes/kr210l150/visual/link_6.dae"/>
-        </geometry>
-        <origin xyz="0 0 0" rpy="0 0 0"/>
-    </visual>
-    <collision>
-        <geometry>
-            <mesh filename="package://kr210_description/meshes/kr210l150/collision/link_6.stl"/>
-        </geometry>
-        <origin xyz="0 0 0" rpy="0 0 0"/>
-    </collision>
-    <!-- <inertial>
+            <mesh filename="file://$(find kr210_description)/meshes/kr210l150/visual/link_6.dae"/>
+        </geometry>
+        <origin xyz="0 0 0" rpy="0 0 0"/>
+    </visual>
+    <collision>
+        <geometry>
+            <mesh filename="file://$(find kr210_description)/meshes/kr210l150/collision/link_6.stl"/>
+        </geometry>
+        <origin xyz="0 0 0" rpy="0 0 0"/>
+    </collision>
+    <inertial>
         <mass value="${mass6}"/>
         <inertia ixx="0.004" ixy="0" ixz="0" iyy="0.003" iyz="0" izz="0.003"/>
         <origin xyz="0 0 0" rpy="0 0 0"/>
-    </inertial> -->
+    </inertial>
 </link>
 <joint name="fixed_base_joint" type="fixed">
@@ -156,4 +165,5 @@
     <axis xyz="0 0 1"/>
     <limit lower="${-185.0 * (pi / 180.0)}" upper="${185.0 * (pi / 180.0)}" effort="300" velocity="${123.0 * (pi / 180.0)}"/>
+    <dynamics friction="1000" damping="1000"/>
 </joint>
 <joint name="joint_2" type="revolute">
@@ -163,4 +173,5 @@
     <axis xyz="0 1 0"/>
     <limit lower="${-45*pi/180}" upper="${85*pi/180}" effort="300" velocity="${115*pi/180}"/>
+    <dynamics friction="1000" damping="1000"/>
 </joint>
 <joint name="joint_3" type="revolute">
@@ -170,4 +181,5 @@
     <axis xyz="0 1 0"/>
     <limit lower="${-210*pi/180}" upper="${65*pi/180}" effort="300" velocity="${112 * pi/180}"/>
+    <dynamics friction="1000" damping="1000"/>
 </joint>
 <joint name="joint_4" type="revolute">
@@ -177,4 +189,5 @@
     <axis xyz="1 0 0"/>
     <limit lower="${-125 * pi/180}" upper="${125*pi/180}" effort="300" velocity="${179*pi/180}"/>
+    <dynamics friction="1000" damping="1000"/>
 </joint>
 <joint name="joint_5" type="revolute">
@@ -184,4 +197,5 @@
     <axis xyz="0 1 0"/>
     <limit lower="${-125 * pi/180}" upper="${125*pi/180}" effort="300" velocity="${172*pi/180}"/>
+    <dynamics friction="1000" damping="1000"/>
 </joint>
 <joint name="joint_6" type="revolute">
@@ -191,4 +205,5 @@
     <axis xyz="1 0 0"/>
     <limit lower="${-350*pi/180}" upper="${350*pi/180}" effort="300" velocity="${219*pi/180}"/>
+    <dynamics friction="1000" damping="1000"/>
 </joint>
 </robot>

Commit message: move the gripper to a seperate file

File: install/kr210_description/share/kr210_description/urdf/kr210.urdf.xacro (robot description, xacro)
@@ -1,5 +1,6 @@
 <?xml version="1.0"?>
 <robot name="kuka" xmlns:xacro="http://www.ros.org/wiki/xacro">
-    <!-- <xacro:include filename="kr210_arm_gazebo.urdf.xacro"/> -->
+    <xacro:include filename="kr210_arm_gazebo.urdf.xacro"/>
     <xacro:include filename="kr210_arm.urdf.xacro"/>
+    <xacro:include filename="kr210_gripper.urdf.xacro"/>
 </robot>

File: install/kr210_description/share/kr210_description/urdf/kr210_arm.urdf.xacro (robot description, xacro)
@@ -8,4 +8,6 @@
 <xacro:property name="mass5" value="7"/>
 <xacro:property name="mass6" value="0.5"/>
+<xacro:property name="gripper_mass" value="0.3"/>
+<xacro:property name="finger_mass" value="0.1"/>
 <link name="base_footprint"/>
 <link name="base_link">
@@ -142,49 +144,4 @@
     </inertial>
 </link>
-<link name="gripper_link">
-    <visual>
-        <geometry>
-            <mesh filename="file://$(find kr210_description)/meshes/gripper/gripper_base.dae"/>
-        </geometry>
-        <origin xyz="0 0 0" rpy="0 0 0"/>
-    </visual>
-</link>
-<link name="right_finger_link">
-    <visual>
-        <geometry>
-            <mesh filename="file://$(find kr210_description)/meshes/gripper/finger_right.dae"/>
-        </geometry>
-        <origin xyz="0 0 0" rpy="0 0 0"/>
-    </visual>
-</link>
-<link name="left_finger_link">
-    <visual>
-        <geometry>
-            <mesh filename="file://$(find kr210_description)/meshes/gripper/finger_left.dae"/>
-        </geometry>
-        <origin xyz="0 0 0" rpy="0 0 0"/>
-    </visual>
-</link>
-<joint name="gripper_joint" type="fixed">
-    <parent link="link_6"/>
-    <child link="gripper_link"/>
-    <origin xyz="0.11 0 0" rpy="0 0 0"/>
-</joint>
-<joint name="gripper_right_finger_joint" type="prismatic">
-    <parent link="gripper_link"/>
-    <child link="right_finger_link"/>
-    <origin xyz="0.15 -0.0725 0" rpy="0 0 0"/>
-    <axis xyz="0 1 0"/>
-    <limit effort="100" lower="-0.01" upper="0.06" velocity="0.05"/>
-    <dynamics damping="0.7"/>
-</joint>
-<joint name="gripper_left_finger_joint" type="prismatic">
-    <parent link="gripper_link"/>
-    <child link="left_finger_link"/>
-    <origin xyz="0.15 0.0725 0" rpy="0 0 0"/>
-    <axis xyz="0 -1 0"/>
-    <limit effort="100" lower="-0.01" upper="0.06" velocity="0.05"/>
-    <dynamics damping="0.7"/>
-</joint>
 <joint name="fixed_base_joint" type="fixed">
     <parent link="base_footprint"/>
@@ -198,5 +155,5 @@
     <axis xyz="0 0 1"/>
     <limit lower="${-185.0 * (pi / 180.0)}" upper="${185.0 * (pi / 180.0)}" effort="300" velocity="${123.0 * (pi / 180.0)}"/>
-    <dynamics friction="1000" damping="1000"/>
+    <!-- <dynamics friction="1000" damping="1000"/> -->
 </joint>
 <joint name="joint_2" type="revolute">
@@ -206,5 +163,5 @@
     <axis xyz="0 1 0"/>
     <limit lower="${-45*pi/180}" upper="${85*pi/180}" effort="300" velocity="${115*pi/180}"/>
-    <dynamics friction="1000" damping="1000"/>
+    <!-- <dynamics friction="1000" damping="1000"/> -->
 </joint>
 <joint name="joint_3" type="revolute">
@@ -214,5 +171,5 @@
     <axis xyz="0 1 0"/>
     <limit lower="${-210*pi/180}" upper="${65*pi/180}" effort="300" velocity="${112 * pi/180}"/>
-    <dynamics friction="1000" damping="1000"/>
+    <!-- <dynamics friction="1000" damping="1000"/> -->
 </joint>
 <joint name="joint_4" type="revolute">
@@ -222,5 +179,5 @@
     <axis xyz="1 0 0"/>
     <limit lower="${-125 * pi/180}" upper="${125*pi/180}" effort="300" velocity="${179*pi/180}"/>
-    <dynamics friction="1000" damping="1000"/>
+    <!-- <dynamics friction="1000" damping="1000"/> -->
 </joint>
 <joint name="joint_5" type="revolute">
@@ -230,5 +187,5 @@
     <axis xyz="0 1 0"/>
     <limit lower="${-125 * pi/180}" upper="${125*pi/180}" effort="300" velocity="${172*pi/180}"/>
-    <dynamics friction="1000" damping="1000"/>
+    <!-- <dynamics friction="1000" damping="1000"/> -->
 </joint>
 <joint name="joint_6" type="revolute">
@@ -238,5 +195,65 @@
     <axis xyz="1 0 0"/>
     <limit lower="${-350*pi/180}" upper="${350*pi/180}" effort="300" velocity="${219*pi/180}"/>
-    <dynamics friction="1000" damping="1000"/>
-</joint>
+    <!-- <dynamics friction="1000" damping="1000"/> -->
+</joint>
+<transmission name="trans_1">
+    <type>transmission_interface/SimpleTransmission</type>
+    <joint name="joint_1">
+        <hardwareInterface>hardware_interface/PositionJointInterface</hardwareInterface>
+    </joint>
+    <actuator name="motor1">
+        <hardwareInterface>hardware_interface/PositionJointInterface</hardwareInterface>
+        <mechanicalReduction>1</mechanicalReduction>
+    </actuator>
+</transmission>
+<transmission name="trans_2">
+    <type>transmission_interface/SimpleTransmission</type>
+    <joint name="joint_2">
+        <hardwareInterface>hardware_interface/PositionJointInterface</hardwareInterface>
+    </joint>
+    <actuator name="motor2">
+        <hardwareInterface>hardware_interface/PositionJointInterface</hardwareInterface>
+        <mechanicalReduction>1</mechanicalReduction>
+    </actuator>
+</transmission>
+<transmission name="trans_3">
+    <type>transmission_interface/SimpleTransmission</type>
+    <joint name="joint_3">
+        <hardwareInterface>hardware_interface/PositionJointInterface</hardwareInterface>
+    </joint>
+    <actuator name="motor3">
+        <hardwareInterface>hardware_interface/PositionJointInterface</hardwareInterface>
+        <mechanicalReduction>1</mechanicalReduction>
+    </actuator>
+</transmission>
+<transmission name="trans_4">
+    <type>transmission_interface/SimpleTransmission</type>
+    <joint name="joint_4">
+        <hardwareInterface>hardware_interface/PositionJointInterface</hardwareInterface>
+    </joint>
+    <actuator name="motor4">
+        <hardwareInterface>hardware_interface/PositionJointInterface</hardwareInterface>
+        <mechanicalReduction>1</mechanicalReduction>
+    </actuator>
+</transmission>
+<transmission name="trans_5">
+    <type>transmission_interface/SimpleTransmission</type>
+    <joint name="joint_5">
+        <hardwareInterface>hardware_interface/PositionJointInterface</hardwareInterface>
+    </joint>
+    <actuator name="motor5">
+        <hardwareInterface>hardware_interface/PositionJointInterface</hardwareInterface>
+        <mechanicalReduction>1</mechanicalReduction>
+    </actuator>
+</transmission>
+<transmission name="trans_6">
+    <type>transmission_interface/SimpleTransmission</type>
+    <joint name="joint_6">
+        <hardwareInterface>hardware_interface/PositionJointInterface</hardwareInterface>
+    </joint>
+    <actuator name="motor6">
+        <hardwareInterface>hardware_interface/PositionJointInterface</hardwareInterface>
+        <mechanicalReduction>1</mechanicalReduction>
+    </actuator>
+</transmission>
 </robot>

File: install/kr210_description/share/kr210_description/urdf/kr210_arm_gazebo.urdf.xacro (robot description, xacro)
@@ -6,3 +6,27 @@
         <mu2>2</mu2>
     </gazebo>
+    <gazebo reference="link_1">
+        <mu1>0.2</mu1>
+        <mu2>0.2</mu2>
+    </gazebo>
+    <gazebo reference="link_2">
+        <mu1>0.2</mu1>
+        <mu2>0.2</mu2>
+    </gazebo>
+     <gazebo reference="link_3">
+        <mu1>0.2</mu1>
+        <mu2>0.2</mu2>
+    </gazebo>
+    <gazebo reference="link_4">
+        <mu1>0.2</mu1>
+        <mu2>0.2</mu2>
+    </gazebo>
+     <gazebo reference="link_5">
+        <mu1>0.2</mu1>
+        <mu2>0.2</mu2>
+    </gazebo>
+    <gazebo reference="link_6">
+        <mu1>0.2</mu1>
+        <mu2>0.2</mu2>
+    </gazebo>
 </robot>
