Commit message: move transmission to seperate file

File: install/kr210_description/share/kr210_description/urdf/kr210.urdf.xacro (robot description, xacro)
@@ -1,6 +1,8 @@
 <?xml version="1.0"?>
 <robot name="kuka" xmlns:xacro="http://www.ros.org/wiki/xacro">
-    <xacro:include filename="kr210_arm_gazebo.urdf.xacro"/>
-    <xacro:include filename="kr210_arm.urdf.xacro"/>
-    <xacro:include filename="kr210_gripper.urdf.xacro"/>
+    <xacro:include filename="kr210_arm.xacro"/>
+    <xacro:include filename="kr210_gripper.xacro"/>
+    <xacro:include filename="kr210_trans.xacro"/>
+    <xacro:include filename="kr210_arm_gazebo.xacro"/>
+    <xacro:include filename="kr210_gripper_gazebo.xacro"/>
 </robot>

File: install/kr210_description/share/kr210_description/urdf/kr210_arm.xacro (robot description, xacro)
@@ -197,63 +197,3 @@
     <dynamics friction="1000" damping="1000"/>
 </joint>
-<transmission name="trans_1">
-    <type>transmission_interface/SimpleTransmission</type>
-    <joint name="joint_1">
-        <hardwareInterface>hardware_interface/PositionJointInterface</hardwareInterface>
-    </joint>
-    <actuator name="motor1">
-        <hardwareInterface>hardware_interface/PositionJointInterface</hardwareInterface>
-        <mechanicalReduction>1</mechanicalReduction>
-    </actuator>
-</transmission>
-<transmission name="trans_2">
-    <type>transmission_interface/SimpleTransmission</type>
-    <joint name="joint_2">
-        <hardwareInterface>hardware_interface/PositionJointInterface</hardwareInterface>
-    </joint>
-    <actuator name="motor2">
-        <hardwareInterface>hardware_interface/PositionJointInterface</hardwareInterface>
-        <mechanicalReduction>1</mechanicalReduction>
-    </actuator>
-</transmission>
-<transmission name="trans_3">
-    <type>transmission_interface/SimpleTransmission</type>
-    <joint name="joint_3">
-        <hardwareInterface>hardware_interface/PositionJointInterface</hardwareInterface>
-    </joint>
-    <actuator name="motor3">
-        <hardwareInterface>hardware_interface/PositionJointInterface</hardwareInterface>
-        <mechanicalReduction>1</mechanicalReduction>
-    </actuator>
-</transmission>
-<transmission name="trans_4">
-    <type>transmission_interface/SimpleTransmission</type>
-    <joint name="joint_4">
-        <hardwareInterface>hardware_interface/PositionJointInterface</hardwareInterface>
-    </joint>
-    <actuator name="motor4">
-        <hardwareInterface>hardware_interface/PositionJointInterface</hardwareInterface>
-        <mechanicalReduction>1</mechanicalReduction>
-    </actuator>
-</transmission>
-<transmission name="trans_5">
-    <type>transmission_interface/SimpleTransmission</type>
-    <joint name="joint_5">
-        <hardwareInterface>hardware_interface/PositionJointInterface</hardwareInterface>
-    </joint>
-    <actuator name="motor5">
-        <hardwareInterface>hardware_interface/PositionJointInterface</hardwareInterface>
-        <mechanicalReduction>1</mechanicalReduction>
-    </actuator>
-</transmission>
-<transmission name="trans_6">
-    <type>transmission_interface/SimpleTransmission</type>
-    <joint name="joint_6">
-        <hardwareInterface>hardware_interface/PositionJointInterface</hardwareInterface>
-    </joint>
-    <actuator name="motor6">
-        <hardwareInterface>hardware_interface/PositionJointInterface</hardwareInterface>
-        <mechanicalReduction>1</mechanicalReduction>
-    </actuator>
-</transmission>
 </robot>

File: src/kr210_description/urdf/kr210_arm.xacro (robot description, xacro)
@@ -155,5 +155,5 @@
     <axis xyz="0 0 1"/>
     <limit lower="${-185.0 * (pi / 180.0)}" upper="${185.0 * (pi / 180.0)}" effort="300" velocity="${123.0 * (pi / 180.0)}"/>
-    <!-- <dynamics friction="1000" damping="1000"/> -->
+    <dynamics friction="1000" damping="1000"/>
 </joint>
 <joint name="joint_2" type="revolute">
@@ -163,5 +163,5 @@
     <axis xyz="0 1 0"/>
     <limit lower="${-45*pi/180}" upper="${85*pi/180}" effort="300" velocity="${115*pi/180}"/>
-    <!-- <dynamics friction="1000" damping="1000"/> -->
+    <dynamics friction="1000" damping="1000"/>
 </joint>
 <joint name="joint_3" type="revolute">
@@ -171,5 +171,5 @@
     <axis xyz="0 1 0"/>
     <limit lower="${-210*pi/180}" upper="${65*pi/180}" effort="300" velocity="${112 * pi/180}"/>
-    <!-- <dynamics friction="1000" damping="1000"/> -->
+    <dynamics friction="1000" damping="1000"/>
 </joint>
 <joint name="joint_4" type="revolute">
@@ -179,5 +179,5 @@
     <axis xyz="1 0 0"/>
     <limit lower="${-125 * pi/180}" upper="${125*pi/180}" effort="300" velocity="${179*pi/180}"/>
-    <!-- <dynamics friction="1000" damping="1000"/> -->
+    <dynamics friction="1000" damping="1000"/>
 </joint>
 <joint name="joint_5" type="revolute">
@@ -187,5 +187,5 @@
     <axis xyz="0 1 0"/>
     <limit lower="${-125 * pi/180}" upper="${125*pi/180}" effort="300" velocity="${172*pi/180}"/>
-    <!-- <dynamics friction="1000" damping="1000"/> -->
+    <dynamics friction="1000" damping="1000"/>
 </joint>
 <joint name="joint_6" type="revolute">
@@ -195,65 +195,5 @@
     <axis xyz="1 0 0"/>
     <limit lower="${-350*pi/180}" upper="${350*pi/180}" effort="300" velocity="${219*pi/180}"/>
-    <!-- <dynamics friction="1000" damping="1000"/> -->
+    <dynamics friction="1000" damping="1000"/>
 </joint>
-<transmission name="trans_1">
-    <type>transmission_interface/SimpleTransmission</type>
-    <joint name="joint_1">
-        <hardwareInterface>hardware_interface/PositionJointInterface</hardwareInterface>
-    </joint>
-    <actuator name="motor1">
-        <hardwareInterface>hardware_interface/PositionJointInterface</hardwareInterface>
-        <mechanicalReduction>1</mechanicalReduction>
-    </actuator>
-</transmission>
-<transmission name="trans_2">
-    <type>transmission_interface/SimpleTransmission</type>
-    <joint name="joint_2">
-        <hardwareInterface>hardware_interface/PositionJointInterface</hardwareInterface>
-    </joint>
-    <actuator name="motor2">
-        <hardwareInterface>hardware_interface/PositionJointInterface</hardwareInterface>
-        <mechanicalReduction>1</mechanicalReduction>
-    </actuator>
-</transmission>
-<transmission name="trans_3">
-    <type>transmission_interface/SimpleTransmission</type>
-    <joint name="joint_3">
-        <hardwareInterface>hardware_interface/PositionJointInterface</hardwareInterface>
-    </joint>
-    <actuator name="motor3">
-        <hardwareInterface>hardware_interface/PositionJointInterface</hardwareInterface>
-        <mechanicalReduction>1</mechanicalReduction>
-    </actuator>
-</transmission>
-<transmission name="trans_4">
-    <type>transmission_interface/SimpleTransmission</type>
-    <joint name="joint_4">
-        <hardwareInterface>hardware_interface/PositionJointInterface</hardwareInterface>
-    </joint>
-    <actuator name="motor4">
-        <hardwareInterface>hardware_interface/PositionJointInterface</hardwareInterface>
-        <mechanicalReduction>1</mechanicalReduction>
-    </actuator>
-</transmission>
-<transmission name="trans_5">
-    <type>transmission_interface/SimpleTransmission</type>
-    <joint name="joint_5">
-        <hardwareInterface>hardware_interface/PositionJointInterface</hardwareInterface>
-    </joint>
-    <actuator name="motor5">
-        <hardwareInterface>hardware_interface/PositionJointInterface</hardwareInterface>
-        <mechanicalReduction>1</mechanicalReduction>
-    </actuator>
-</transmission>
-<transmission name="trans_6">
-    <type>transmission_interface/SimpleTransmission</type>
-    <joint name="joint_6">
-        <hardwareInterface>hardware_interface/PositionJointInterface</hardwareInterface>
-    </joint>
-    <actuator name="motor6">
-        <hardwareInterface>hardware_interface/PositionJointInterface</hardwareInterface>
-        <mechanicalReduction>1</mechanicalReduction>
-    </actuator>
-</transmission>
 </robot>

File: src/kr210_description/urdf/kr210_gripper.xacro (robot description, xacro)
@@ -79,23 +79,3 @@
         <dynamics damping="0.7"/>
     </joint>
-    <transmission name="trans_7">
-        <type>transmission_interface/SimpleTransmission</type>
-        <joint name="gripper_right_finger_joint">
-            <hardwareInterface>hardware_interface/EffortJointInterface</hardwareInterface>
-        </joint>
-        <actuator name="motor_7">
-            <hardwareInterface>hardware_interface/EffortJointInterface</hardwareInterface>
-            <mechanicalReduction>1</mechanicalReduction>
-        </actuator>
-    </transmission>
-    <transmission name="trans_8">
-        <type>transmission_interface/SimpleTransmission</type>
-        <joint name="gripper_left_finger_joint">
-            <hardwareInterface>hardware_interface/EffortJointInterface</hardwareInterface>
-        </joint>
-        <actuator name="motor_8">
-            <hardwareInterface>hardware_interface/EffortJointInterface</hardwareInterface>
-            <mechanicalReduction>1</mechanicalReduction>
-        </actuator>
-    </transmission>
 </robot>
