Commit message: remove base footprint

File: kr210_description/urdf/kr210_arm.xacro (robot description, xacro)
@@ -10,5 +10,5 @@
 <xacro:property name="gripper_mass" value="0.3"/>
 <xacro:property name="finger_mass" value="0.1"/>
-<link name="base_footprint"/>
+<!-- <link name="base_footprint"/> -->
 <link name="base_link">
     <visual>
@@ -144,9 +144,9 @@
     </inertial>
 </link>
-<joint name="fixed_base_joint" type="fixed">
+<!-- <joint name="fixed_base_joint" type="fixed">
     <parent link="base_footprint"/>
     <child link="base_link"/>
     <origin xyz="0 0 0" rpy="0 0 0"/>
-</joint>
+</joint> -->
 <joint name="joint_1" type="revolute">
     <parent link="base_link"/>

Commit message: add gazebo launch file

File: kr210_description/urdf/kr210_arm.xacro (robot description, xacro)
@@ -10,5 +10,5 @@
 <xacro:property name="gripper_mass" value="0.3"/>
 <xacro:property name="finger_mass" value="0.1"/>
-<!-- <link name="base_footprint"/> -->
+<link name="world"/>
 <link name="base_link">
     <visual>
@@ -26,5 +26,5 @@
     <inertial>
         <mass value="${base_mass}"/>
-        <inertia ixx="60" iyy="0" izz="0" ixy="70" ixz="0" iyz="100" />
+        <inertia ixx="60" ixy="0" ixz="0" iyy="70" iyz="0" izz="100" />
         <origin xyz="0 0 0" rpy="0 0 0"/>
     </inertial>
@@ -144,9 +144,9 @@
     </inertial>
 </link>
-<!-- <joint name="fixed_base_joint" type="fixed">
-    <parent link="base_footprint"/>
+<joint name="fixed_base_joint" type="fixed">
+    <parent link="world"/>
     <child link="base_link"/>
     <origin xyz="0 0 0" rpy="0 0 0"/>
-</joint> -->
+</joint>
 <joint name="joint_1" type="revolute">
     <parent link="base_link"/>

File: kr210_description/urdf/kr210_gripper.xacro (robot description, xacro)
@@ -36,5 +36,5 @@
             <mass value="${finger_mass}"/>
             <origin xyz="0 0 0" rpy="0 0 0"/>
-            <inertia ixx="0.002" ixy="0" ixz="0" iyy="0.0002" iyz="0" izz="0.0002"/>
+            <inertia ixx="0.0002" ixy="0" ixz="0" iyy="0.0002" iyz="0" izz="0.0002"/>
         </inertial>
     </link>
@@ -55,5 +55,5 @@
             <mass value="${finger_mass}"/>
             <origin xyz="0 0 0" rpy="0 0 0"/>
-            <inertia ixx="0.002" ixy="0" ixz="0" iyy="0.0002" iyz="0" izz="0.0002"/>
+            <inertia ixx="0.0002" ixy="0" ixz="0" iyy="0.0002" iyz="0" izz="0.0002"/>
         </inertial>
     </link>

Commit message: run all function from a single launch file

File: kr210_description/urdf/kr210_arm.xacro (robot description, xacro)
@@ -10,5 +10,5 @@
 <xacro:property name="gripper_mass" value="0.03"/>
 <xacro:property name="finger_mass" value="0.01"/>
-<!-- <link name="world"/> -->
+<link name="world"/>
 <link name="base_link">
     <visual>
@@ -144,9 +144,9 @@
     </inertial>
 </link>
-<!-- <joint name="fixed_base_joint" type="fixed">
+<joint name="fixed_base_joint" type="fixed">
     <parent link="world"/>
     <child link="base_link"/>
     <origin xyz="0 0 0" rpy="0 0 0"/>
-</joint> -->
+</joint>
 <joint name="joint_1" type="revolute">
     <parent link="base_link"/>
