Commit message: create simple node to interact with moveit api

File: kr210_description/urdf/kr210_gripper.xacro (robot description, xacro)
@@ -1,4 +1,7 @@
 <?xml version="1.0"?>
 <robot>
+    <material name="grey">
+        <color rgba="0.4 0.4 0.4 1"/>
+    </material>
     <link name="gripper_link">
         <visual>
@@ -7,4 +10,5 @@
             </geometry>
             <origin xyz="0 0 0" rpy="0 0 0"/>
+            <material name="grey"/>
         </visual>
         <collision>
@@ -26,4 +30,5 @@
             </geometry>
             <origin xyz="0 0 0" rpy="0 0 0"/>
+            <material name="grey"/>
         </visual>
         <collision>
@@ -45,4 +50,5 @@
             </geometry>
             <origin xyz="0 0 0" rpy="0 0 0"/>
+            <material name="grey"/>
         </visual>
         <collision>
