Commit message: move the robot in gazebo fix some bugs

File: kr210_description/urdf/kr210.urdf.xacro (robot description, xacro)
@@ -3,7 +3,7 @@
     <xacro:include filename="kr210_arm.xacro"/>
     <xacro:include filename="kr210_gripper.xacro"/>
-    <xacro:include filename="kr210_trans.xacro"/>
+    <!-- <xacro:include filename="kr210_trans.xacro"/> -->
     <xacro:include filename="kr210_arm_gazebo.xacro"/>
-    <xacro:include filename="kr210_gripper_gazebo.xacro"/>
+    <!-- <xacro:include filename="kr210_gripper_gazebo.xacro"/> -->
     <xacro:include filename="kr210_ros2_control.xacro"/>
 </robot>

File: kr210_description/urdf/kr210_arm.xacro (robot description, xacro)
@@ -1,14 +1,14 @@
 <?xml version="1.0"?>
 <robot xmlns:xacro="http://www.ros.org/wiki/xacro">
-<xacro:property name="base_mass" value="150"/>
-<xacro:property name="mass1" value="138"/>
-<xacro:property name="mass2" value="95"/>
-<xacro:property name="mass3" value="71"/>
-<xacro:property name="mass4" value="17"/>
-<xacro:property name="mass5" value="7"/>
-<xacro:property name="mass6" value="0.5"/>
-<xacro:property name="gripper_mass" value="0.3"/>
-<xacro:property name="finger_mass" value="0.1"/>
-<link name="world"/>
+<xacro:property name="base_mass" value="15"/>
+<xacro:property name="mass1" value="13.8"/>
+<xacro:property name="mass2" value="9.5"/>
+<xacro:property name="mass3" value="7.1"/>
+<xacro:property name="mass4" value="1.7"/>
+<xacro:property name="mass5" value="0.7"/>
+<xacro:property name="mass6" value="0.05"/>
+<xacro:property name="gripper_mass" value="0.03"/>
+<xacro:property name="finger_mass" value="0.01"/>
+<!-- <link name="world"/> -->
 <link name="base_link">
     <visual>
@@ -26,5 +26,5 @@
     <inertial>
         <mass value="${base_mass}"/>
-        <inertia ixx="60" ixy="0" ixz="0" iyy="70" iyz="0" izz="100" />
+        <inertia ixx="6" ixy="0" ixz="0" iyy="7" iyz="0" izz="10" />
         <origin xyz="0 0 0" rpy="0 0 0"/>
     </inertial>
@@ -45,5 +45,5 @@
     <inertial>
         <mass value="${mass1}"/>
-        <inertia ixx="30" ixy="0" ixz="0" iyy="50" iyz="0" izz="50"/>
+        <inertia ixx="3" ixy="0" ixz="0" iyy="5" iyz="0" izz="5"/>
         <origin xyz="0 0 0.4" rpy="0 0 0"/>
     </inertial>
@@ -64,5 +64,5 @@
     <inertial>
         <mass value="${mass2}"/>
-        <inertia ixx="40" ixy="0" ixz="0" iyy="40" iyz="0" izz="10"/>
+        <inertia ixx="4" ixy="0" ixz="0" iyy="4" iyz="0" izz="1"/>
         <origin xyz="0 0 0" rpy="0 0 0"/>
     </inertial>
@@ -83,5 +83,5 @@
     <inertial>
         <mass value="${mass3}"/>
-        <inertia ixx="1" ixy="0" ixz="0" iyy="10" iyz="0" izz="10"/>
+        <inertia ixx="0.1" ixy="0" ixz="0" iyy="1" iyz="0" izz="1"/>
         <origin xyz="0.18842 0.18344 -0.042799" rpy="0 0 0"/>
     </inertial>
@@ -102,5 +102,5 @@
     <inertial>
         <mass value="${mass4}"/>
-        <inertia ixx="0.18" ixy="0" ixz="0" iyy="0.55" iyz="0" izz="0.64"/>
+        <inertia ixx="0.018" ixy="0" ixz="0" iyy="0.055" iyz="0" izz="0.064"/>
         <origin xyz="0.27146 -0.007326 0" rpy="0 0 0"/>
     </inertial>
@@ -121,5 +121,5 @@
     <inertial>
         <mass value="${mass5}"/>
-        <inertia ixx="0.04" ixy="0" ixz="0" iyy="0.068" iyz="0" izz="0.068"/>
+        <inertia ixx="0.004" ixy="0" ixz="0" iyy="0.0068" iyz="0" izz="0.0068"/>
         <origin xyz="0 0 0" rpy="0 0 0"/>
     </inertial>
@@ -140,13 +140,13 @@
     <inertial>
         <mass value="${mass6}"/>
-        <inertia ixx="0.004" ixy="0" ixz="0" iyy="0.003" iyz="0" izz="0.003"/>
+        <inertia ixx="0.0004" ixy="0" ixz="0" iyy="0.0003" iyz="0" izz="0.0003"/>
         <origin xyz="0 0 0" rpy="0 0 0"/>
     </inertial>
 </link>
-<joint name="fixed_base_joint" type="fixed">
+<!-- <joint name="fixed_base_joint" type="fixed">
     <parent link="world"/>
     <child link="base_link"/>
     <origin xyz="0 0 0" rpy="0 0 0"/>
-</joint>
+</joint> -->
 <joint name="joint_1" type="revolute">
     <parent link="base_link"/>
@@ -155,5 +155,5 @@
     <axis xyz="0 0 1"/>
     <limit lower="${-185.0 * (pi / 180.0)}" upper="${185.0 * (pi / 180.0)}" effort="300" velocity="${123.0 * (pi / 180.0)}"/>
-    <dynamics friction="1000" damping="1000"/>
+    <dynamics friction="0" damping="10"/>
 </joint>
 <joint name="joint_2" type="revolute">
@@ -163,5 +163,5 @@
     <axis xyz="0 1 0"/>
     <limit lower="${-45*pi/180}" upper="${85*pi/180}" effort="300" velocity="${115*pi/180}"/>
-    <dynamics friction="1000" damping="1000"/>
+    <dynamics friction="0" damping="10"/>
 </joint>
 <joint name="joint_3" type="revolute">
@@ -170,6 +170,6 @@
     <origin xyz="0 0 1.25" rpy="0 0 0"/>
     <axis xyz="0 1 0"/>
-    <limit lower="${-210*pi/180}" upper="${65*pi/180}" effort="300" velocity="${112 * pi/180}"/>
-    <dynamics friction="1000" damping="1000"/>
+    <limit lower="${-210*pi/180}" upper="${65*pi/180}" effort="3000" velocity="${112 * pi/180}"/>
+    <dynamics friction="0" damping="10"/>
 </joint>
 <joint name="joint_4" type="revolute">
@@ -178,6 +178,6 @@
     <origin xyz="0.96 0 -0.054" rpy="0 0 0"/>
     <axis xyz="1 0 0"/>
-    <limit lower="${-125 * pi/180}" upper="${125*pi/180}" effort="300" velocity="${179*pi/180}"/>
-    <dynamics friction="1000" damping="1000"/>
+    <limit lower="${-125 * pi/180}" upper="${125*pi/180}" effort="3000" velocity="${179*pi/180}"/>
+    <dynamics friction="0" damping="10"/>
 </joint>
 <joint name="joint_5" type="revolute">
@@ -186,6 +186,6 @@
     <origin xyz="0.54 0 0" rpy="0 0 0"/>
     <axis xyz="0 1 0"/>
-    <limit lower="${-125 * pi/180}" upper="${125*pi/180}" effort="300" velocity="${172*pi/180}"/>
-    <dynamics friction="1000" damping="1000"/>
+    <limit lower="${-125 * pi/180}" upper="${125*pi/180}" effort="3000" velocity="${172*pi/180}"/>
+    <dynamics friction="0" damping="10"/>
 </joint>
 <joint name="joint_6" type="revolute">
@@ -194,6 +194,6 @@
     <origin xyz="0.193 0 0" rpy="0 0 0"/>
     <axis xyz="1 0 0"/>
-    <limit lower="${-350*pi/180}" upper="${350*pi/180}" effort="300" velocity="${219*pi/180}"/>
-    <dynamics friction="1000" damping="1000"/>
+    <limit lower="${-350*pi/180}" upper="${350*pi/180}" effort="3000" velocity="${219*pi/180}"/>
+    <dynamics friction="0" damping="10"/>
 </joint>
 </robot>

File: kr210_description/urdf/kr210_arm_gazebo.xacro (robot description, xacro)
@@ -1,5 +1,5 @@
 <?xml version="1.0"?>
 <robot>
-    <gazebo reference="base_link">
+    <!-- <gazebo reference="base_link">
         <material>Gazebo/Grey</material>
         <mu1>2</mu1>
@@ -29,5 +29,5 @@
         <mu1>0.2</mu1>
         <mu2>0.2</mu2>
-    </gazebo>
+    </gazebo> -->
      <gazebo>
         <plugin filename="ign_ros2_control-system" name="ign_ros2_control::IgnitionROS2ControlPlugin">

Commit message: add object to grasp

File: kr210_description/urdf/kr210.urdf.xacro (robot description, xacro)
@@ -5,5 +5,5 @@
     <!-- <xacro:include filename="kr210_trans.xacro"/> -->
     <xacro:include filename="kr210_arm_gazebo.xacro"/>
-    <!-- <xacro:include filename="kr210_gripper_gazebo.xacro"/> -->
+    <xacro:include filename="kr210_gripper_gazebo.xacro"/>
     <xacro:include filename="kr210_ros2_control.xacro"/>
 </robot>

File: kr210_description/urdf/kr210_gripper.xacro (robot description, xacro)
@@ -75,5 +75,5 @@
         <axis xyz="0 1 0"/>
         <limit effort="100" lower="-0.01" upper="0.06" velocity="0.05"/>
-        <dynamics damping="0.7"/>
+        <dynamics damping="5.0" friction="0.5"/>
     </joint>
     <joint name="gripper_left_finger_joint" type="prismatic">
@@ -83,5 +83,5 @@
         <axis xyz="0 -1 0"/>
         <limit effort="100" lower="-0.01" upper="0.06" velocity="0.05"/>
-        <dynamics damping="0.7"/>
+        <dynamics damping="5.0" friction="0.5"/>
     </joint>
 </robot>

File: kr210_description/urdf/kr210_gripper_gazebo.xacro (robot description, xacro)
@@ -2,10 +2,10 @@
 <robot>
     <gazebo reference="gripper_link">
-        <material>Gazebo/Grey</material>
+        <!-- <material>Gazebo/Grey</material> -->
         <mu1>0.2</mu1>
         <mu2>0.2</mu2>
     </gazebo>
     <gazebo reference="right_finger_link">
-        <material>Gazebo/Grey</material>
+        <!-- <material>Gazebo/Grey</material> -->
         <kp>1000000.0</kp>
         <kd>1.0</kd>
@@ -14,5 +14,5 @@
     </gazebo>
     <gazebo reference="left_finger_link">
-        <material>Gazebo/Grey</material>
+        <!-- <material>Gazebo/Grey</material> -->
         <kp>1000000.0</kp>
         <kd>1.0</kd>
